File: ecad/pcb-pami/pcb-pami.kicad_sch (KiCad schematic)
At the start: 80 parts, among them J1 USB_C_Receptacle_USB2.0_16P, J10 Conn_01x02_Pin, J11 Conn_01x05_Pin, J12 Conn_01x02_Pin, J13 Conn_01x04_Pin, J14 Conn_01x04_Pin, J15 Conn_01x02_Pin, J16 Conn_01x05_Pin, J17 Conn_01x07_Pin, J2 Conn_01x11_Socket, J21 Conn_01x05_Pin, J22 Conn_01x04_Pin, J23 Conn_01x03_Pin, J26 Conn_01x03_Pin, J27 Conn_01x02_Pin, J3 Conn_01x08_Socket, J4 Conn_01x11_Socket, J5 Conn_01x02_Pin, J6 Conn_01x02_Pin, J7 Conn_01x02_Pin, J8 Conn_01x03_Pin, J9 Conn_01x02_Pin, SW1 SW_Push, SW2 SW_Push, U10 MCP23008-xSO, U2 LTC4412xS6, U3 LTC4412xS6, U4 AMS1117-3.3 (UMW), U6 ESP32-S3-WROOM-1, U7 TMC2209_SILENTSTEPSTICK, U8 TMC2209_SILENTSTEPSTICK, U9 TMC2209_SILENTSTEPSTICK

Commit message: [ECAD] debut nouvelle carte, [FW] generation strat web
Parts:
- removed AS1, AS2, J13: Conn_01x04_Pin, Connector_PinHeader_2.54mm:PinHeader_1x04_P2.54mm_Vertical, symbol Connector:Conn_01x04_Pin
- removed C3: 100u, Capacitor_THT:C_Radial_D8.0mm_H11.5mm_P3.50mm, symbol Device:C_Polarized_Small
- removed C8: 470u, Capacitor_THT:C_Radial_D8.0mm_H11.5mm_P3.50mm, symbol Device:C_Polarized_Small
- removed U7: TMC2209_SILENTSTEPSTICK, TMC2209:MODULE_TMC2209_SILENTSTEPSTICK, symbol TMC2209_SILENTSTEPSTICK:TMC2209_SILENTSTEPSTICK
Connections:
- net DIR3: no longer U6.20 (IO12)
- net STEP3: no longer U6.19 (IO11)
Other:
- moved on the sheet: C16
